File: kicad/Picopede/Picopede.kicad_sch (KiCad schematic)
At the start: 49 parts, among them J1 USB_B_Micro, J2 Conn_02x26_Odd_Even, J3 Conn_02x26_Odd_Even, J4 SM03B-SRSS-TB, SW1 SW_Push, SW2 SW_Push, U1 RP2350_80QFN, U2 NCP1117-3.3_SOT223, U3 W25Q128JVS, U4 DNF, Y1 ABM8-272-T3

Commit message: made first iteration of the schematic
Parts:
- removed C1, C5: 10u, Capacitor_SMD:C_0805_2012Metric, symbol Device:C
- removed J1: USB_B_Micro, Connector_USB:USB_Micro-B_Amphenol_10103594-0001LF_Horizontal, symbol Connector:USB_B_Micro
- removed J2, J3: Conn_02x26_Odd_Even, Connector_PinHeader_2.54mm:PinHeader_2x26_P2.54mm_Vertical, symbol Connector_Generic:Conn_02x26_Odd_Even
- removed J4: SM03B-SRSS-TB, Connector_JST:JST_SH_SM03B-SRSS-TB_1x03-1MP_P1.00mm_Horizontal, symbol Connector_Generic_MountingPin:Conn_01x03_MountingPin
- removed U2: NCP1117-3.3_SOT223, Package_TO_SOT_SMD:SOT-223-3_TabPin2, symbol Regulator_Linear:NCP1117-3.3_SOT223
- added C23, C24: 10u, Capacitor_SMD:C_0805_2012Metric, symbol Device:C
- added D1, D2: LED, symbol Device:LED
- added J1: USB_C_Plug_USB2.0, symbol Connector:USB_C_Plug_USB2.0
- added J2, J3: Conn_01x32, symbol Connector_Generic:Conn_01x32
- added J5, J6: Conn_01x04, symbol Connector_Generic:Conn_01x04
- added R12, R5: 470, symbol Device:R
- added R14: 1k, symbol Device:R
- added SW3: SW_Push, Button_Switch_SMD:SW_Push_1P1T_NO_Vertical_Wuerth_434133025816, symbol Switch:SW_Push
- added U5: NCP1117-3.3_SOT223, Package_TO_SOT_SMD:SOT-223-3_TabPin2, symbol Regulator_Linear:NCP1117-3.3_SOT223
Connections:
- net +3V3: now also C24.1, J3.3 (Pin_3), J3.4 (Pin_4), J5.1 (Pin_1), R5.1, U5.2 (VO)
- net GND: now also C23.2, C24.2, D1.1 (K), D2.1 (K), J1.A1 (GND), J1.A12 (GND), J1.B1 (GND), J1.B12 (GND), J1.S1 (SHIELD), J2.13 (Pin_13), J2.18 (Pin_18), J2.23 (Pin_23), J2.28 (Pin_28), J2.3 (Pin_3), J2.8 (Pin_8), J3.17 (Pin_17), J3.28 (Pin_28), J3.5 (Pin_5), J3.8 (Pin_8), J5.2 (Pin_2), J6.4 (Pin_4), R14.1, U5.1 (GND)
- net GPIO0: now also J2.1 (Pin_1)
- net GPIO1: now also J2.2 (Pin_2)
- net GPIO10: now also J2.14 (Pin_14)
- net GPIO11: now also J2.15 (Pin_15)
- net GPIO12: now also J2.16 (Pin_16)
- net GPIO13: now also J2.17 (Pin_17)
- net GPIO14: now also J2.19 (Pin_19)
- net GPIO15: now also J2.20 (Pin_20)
- net GPIO16: now also J2.21 (Pin_21)
- net GPIO17: now also J2.22 (Pin_22)
- net GPIO18: now also J2.24 (Pin_24)
- net GPIO19: now also J2.25 (Pin_25)
- net GPIO2: now also J2.4 (Pin_4)
- net GPIO20: now also J2.26 (Pin_26)
- net GPIO21: now also J2.27 (Pin_27)
- net GPIO22: now also J2.29 (Pin_29)
- net GPIO23: now also J2.30 (Pin_30), SW3.1
- net GPIO24: now also J2.31 (Pin_31)
- net GPIO25: now also J2.32 (Pin_32), R12.1
- net GPIO26: now also J3.32 (Pin_32)
- net GPIO27: now also J3.31 (Pin_31)
- net GPIO28: now also J3.30 (Pin_30)
- net GPIO29: now also J3.29 (Pin_29)
- net GPIO3: now also J2.5 (Pin_5)
- net GPIO30: now also J3.27 (Pin_27)
- net GPIO31: now also J3.26 (Pin_26)
- net GPIO32: now also J3.25 (Pin_25)
- net GPIO33: now also J3.24 (Pin_24)
- net GPIO34: now also J3.23 (Pin_23)
- net GPIO35: now also J3.22 (Pin_22)
- net GPIO36: now also J3.21 (Pin_21)
- net GPIO37: now also J3.20 (Pin_20)
- net GPIO38: now also J3.19 (Pin_19)
- net GPIO39: now also J3.18 (Pin_18)
- net GPIO4: now also J2.6 (Pin_6)
- net GPIO40_ADC0: now also J3.16 (Pin_16)
- net GPIO41_ADC1: now also J3.15 (Pin_15)
- net GPIO42_ADC2: now also J3.14 (Pin_14)
- net GPIO43_ADC3: now also J3.13 (Pin_13)
- net GPIO44_ADC4: now also J3.12 (Pin_12)
- net GPIO45_ADC5: now also J3.11 (Pin_11)
- net GPIO46_ADC6: now also J3.10 (Pin_10)
- net GPIO47_ADC7: now also J3.9 (Pin_9)
- net GPIO5: now also J2.7 (Pin_7)
- net GPIO6: now also J2.9 (Pin_9)
- net GPIO7: now also J2.10 (Pin_10)
- net GPIO8: now also J2.11 (Pin_11)
- net GPIO9: now also J2.12 (Pin_12)
- net RUN: now also J3.7 (Pin_7)
- net SWCLK: now also J5.3 (Pin_3)
- net SWD: now also J5.4 (Pin_4)
- net USB_D+: now also J1.A6 (D+)
- net USB_D-: now also J1.A7 (D-)
- net VBUS: now also C23.1, J1.A4 (VBUS), J1.A9 (VBUS), J1.B4 (VBUS), J1.B9 (VBUS), J3.1 (Pin_1), J3.2 (Pin_2), J6.1 (Pin_1), U5.3 (VI)
- new net: D1.2 (A), R12.2
- new net: D2.2 (A), R5.2
- new net: J1.A5 (CC), J1.B5 (VCONN)
- new net: R14.2, SW3.2
- new net 3V3_EN: J3.6 (Pin_6)
- new net USB D+: J6.3 (Pin_3)
- new net USB D-: J6.2 (Pin_2)
Other:
- note added: "Debug Header"
- note added: "USB Header"
- note removed: "JST Debug Connector"
- moved on the sheet: C19
