File: kicad/Picopede/Picopede.kicad_sch (KiCad schematic)
At the start: 56 parts, among them J1 USB_C_Plug_USB2.0, J2 Conn_01x32, J3 Conn_01x32, J5 Conn_01x04, J6 Conn_01x04, SW1 SW_Push, SW2 SW_Push, SW3 SW_Push, U1 RP2350_80QFN, U3 W25Q128JVS, U4 DNF, U5 NCP1117-3.3_SOT223, Y1 ABM8-272-T3

Commit message: finished first version of schematic
Parts:
- removed J1: USB_C_Plug_USB2.0, symbol Connector:USB_C_Plug_USB2.0
- removed U5: NCP1117-3.3_SOT223, Package_TO_SOT_SMD:SOT-223-3_TabPin2, symbol Regulator_Linear:NCP1117-3.3_SOT223
- added D3: B5819W, Diode_SMD:D_SOD-123, symbol Device:D_Schottky
- added J4: USB_C_Receptacle_USB2.0_16P, symbol Connector:USB_C_Receptacle_USB2.0_16P
- added JP2: VREF, Jumper:SolderJumper-2_P1.3mm_Open_TrianglePad1.0x1.5mm, symbol Jumper:Jumper_2_Bridged
- added R15: 470, symbol Device:R
- added R5.1K (x2): 33, Resistor_SMD:R_0402_1005Metric, symbol Device:R
- added U2: AMS1117-3.3, Package_TO_SOT_SMD:SOT-223-3_TabPin2, symbol Regulator_Linear:AMS1117-3.3
- added U5: LM4040DBZ-3, Package_TO_SOT_SMD:SOT-23, symbol Reference_Voltage:LM4040DBZ-3
- C19: value 10u -> 10n C0G; footprint Capacitor_SMD:C_0805_2012Metric -> Capacitor_SMD:C_0603_1608Metric_Pad1.08x0.95mm_HandSolder; LCSC (none) -> C76599; P/N (none) -> C1608C0G1H103JT000N
- C23: value 10u -> 2.2u
- C3, C4: value 15p -> 12p
- R1, R13: value DNF -> 10K
- R11: value DNF -> 0R
Connections:
- net +3V3: now also R15.2, U2.2 (VO); no longer C19.1
- net GND: now also J4.A1 (GND), J4.A12 (GND), J4.B1 (GND), J4.B12 (GND), J4.SH (SHIELD), R5.1K.1, R5.1K.1, U2.1 (GND), U5.2 (A)
- net USB_D+: now also J4.A6 (D+), J4.B6 (D+)
- net USB_D-: now also J4.A7 (D-), J4.B7 (D-)
- net VBUS: now also D3.2 (A), J4.A4 (VBUS), J4.A9 (VBUS), J4.B4 (VBUS), J4.B9 (VBUS); no longer C23.1, J3.2 (Pin_2)
- new net +5VD: C23.1, D3.1 (K), J3.2 (Pin_2), U2.3 (VI)
- new net 3V0_VREF: JP2.2 (B), R15.1, U5.1 (K)
- new net ADC_VREF: C19.1, JP2.1 (A)
- new net USB_CC1: J4.A5 (CC1), R5.1K.2
- new net USB_CC2: J4.B5 (CC2), R5.1K.2
- no-connect marks 1 -> 2
Other:
- note added: "RP2350B"
- note added: "USB-C Interface"
- moved on the sheet: C10, C11, C12, C13, C14, C15, C16, C17, C18, C2, C20, C21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

Commit message: cleaned up schematic
Parts:
- C22: value DNF -> 100n
- R16, R17: renamed from R5.1K; value 33 -> 5.1K
- R9: value DNF -> 0R
- renumbered J2 to J1, J3 to J2, J5 to J3, J6 to J4
Changed lines of the file:
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@@
 			)
 		)
-		(property "Value" "DNF"
+		(property "Value" "100n"
 			(at 79.121 316.103 0)
 			(show_name no)
@@
 		(in_pos_files yes)
 		(dnp no)
-		(property "Reference" "R5.1K"
+		(property "Reference" "R16"
 			(at 89.662 51.9684 0)
 			(show_name no)
@@
 			)
 		)
-		(property "Value" "33"
+		(property "Value" "5.1K"
 			(at 89.662 49.657 0)
 			(show_name no)
@@
 			(project "Picopede"
 				(path "/4d566cad-fdcf-4087-b2b1-2acaa8d49b4f"
-					(reference "R5.1K")
+					(reference "R16")
 					(unit 1)
 				)
@@
 			)
 		)
-		(property "Value" "DNF"
+		(property "Value" "0R"
 			(at 38.608 256.032 0)
 			(show_name no)
@@
 		(dnp no)
 		(fields_autoplaced yes)
-		(property "Reference" "J6"
+		(property "Reference" "J4"
 			(at 544.83 148.5899 0)
 			(show_name no)
@@
 			(project "Picopede"
 				(path "/4d566cad-fdcf-4087-b2b1-2acaa8d49b4f"
-					(reference "J6")
+					(reference "J4")
 					(unit 1)
 				)
@@
 		(dnp no)
 		(fields_autoplaced yes)
-		(property "Reference" "J5"
+		(property "Reference" "J3"
 			(at 500.38 148.5899 0)
 			(show_name no)
@@
 			(project "Picopede"
 				(path "/4d566cad-fdcf-4087-b2b1-2acaa8d49b4f"
-					(reference "J5")
+					(reference "J3")
 					(unit 1)
 				)
@@
 		(in_pos_files yes)
 		(dnp no)
-		(property "Reference" "R5.1K"
+		(property "Reference" "R17"
 			(at 99.822 51.9684 0)
 			(show_name no)
@@
 			)
 		)
-		(property "Value" "33"
+		(property "Value" "5.1K"
 			(at 99.822 49.657 0)
 			(show_name no)
@@
 			(project "Picopede"
 				(path "/4d566cad-fdcf-4087-b2b1-2acaa8d49b4f"
-					(reference "R5.1K")
+					(reference "R17")
 					(unit 1)
 				)
@@
 		(dnp no)
 		(fields_autoplaced yes)
-		(property "Reference" "J2"
+		(property "Reference" "J1"
 			(at 499.11 76.1999 0)
 			(show_name no)
@@
 			(project "Picopede"
 				(path "/4d566cad-fdcf-4087-b2b1-2acaa8d49b4f"
-					(reference "J2")
+					(reference "J1")
 					(unit 1)
 				)
@@
 		(dnp no)
 		(fields_autoplaced yes)
-		(property "Reference" "J3"
+		(property "Reference" "J2"
 			(at 525.78 76.1999 0)
 			(show_name no)
@@
 			(project "Picopede"
 				(path "/4d566cad-fdcf-4087-b2b1-2acaa8d49b4f"
-					(reference "J3")
+					(reference "J2")
 					(unit 1)
 				)

Commit message: header foodprints
Parts:
- renumbered C24 to C1, C23 to C5, J4 to J1, J1 to J2, J2 to J3, J3 to J4, J4 to J5
Connections:
- net +3V3: now also J3.5 (Pin_5); no longer J3.3 (Pin_3)
- net GND: now also J3.3 (Pin_3); no longer J3.5 (Pin_5)
Changed lines of the file:
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@@
 	)
 	(junction
-		(at 551.18 55.88)
-		(diameter 0)
-		(color 0 0 0 0)
-	)
-	(junction
 		(at 48.26 388.62)
 		(diameter 0)
@@
 	)
 	(junction
-		(at 566.42 43.18)
-		(diameter 0)
-		(color 0 0 0 0)
-	)
-	(junction
 		(at 64.77 181.61)
 		(diameter 0)
@@
 	)
 	(junction
+		(at 566.42 45.72)
+		(diameter 0)
+		(color 0 0 0 0)
+	)
+	(junction
 		(at 194.31 104.14)
 		(diameter 0)
@@
 	(wire
 		(pts
+			(xy 566.42 45.72) (xy 566.42 48.26)
+		)
+		(stroke
+			(width 0)
+			(type default)
+		)
+	)
+	(wire
+		(pts
 			(xy 261.62 69.85) (xy 261.62 90.17)
 		)
@@
 	(wire
 		(pts
+			(xy 533.4 43.18) (xy 551.18 43.18)
+		)
+		(stroke
+			(width 0)
+			(type default)
+		)
+	)
+	(wire
+		(pts
 			(xy 85.09 274.32) (xy 97.79 274.32)
 		)
@@
 	(wire
 		(pts
-			(xy 533.4 43.18) (xy 566.42 43.18)
-		)
-		(stroke
-			(width 0)
-			(type default)
-		)
-	)
-	(wire
-		(pts
 			(xy 321.31 133.35) (xy 336.55 133.35)
 		)
@@
 	(wire
 		(pts
-			(xy 566.42 45.72) (xy 566.42 43.18)
+			(xy 566.42 33.02) (xy 566.42 45.72)
 		)
 		(stroke
@@
 	(wire
 		(pts
-			(xy 566.42 43.18) (xy 566.42 33.02)
-		)
-		(stroke
-			(width 0)
-			(type default)
-		)
-	)
-	(wire
-		(pts
 			(xy 284.48 250.19) (xy 284.48 252.73)
 		)
@@
 	(wire
 		(pts
-			(xy 533.4 48.26) (xy 551.18 48.26)
+			(xy 533.4 48.26) (xy 566.42 48.26)
 		)
 		(stroke
@@
 	(wire
 		(pts
-			(xy 551.18 48.26) (xy 551.18 55.88)
-		)
-		(stroke
-			(width 0)
-			(type default)
-		)
-	)
-	(wire
-		(pts
 			(xy 210.82 173.99) (xy 214.63 173.99)
 		)
@@
 		)
 	)
-	(label "GND"
+	(label "3V3"
 		(at 548.64 48.26 180)
 		(effects
@@
 		)
 	)
-	(label "3V3"
+	(label "GND"
 		(at 548.64 43.18 180)
 		(effects
@@
 	)
 	(symbol
+		(lib_name "GND_4")
+		(lib_id "power:GND")
+		(at 551.18 43.18 90)
+		(unit 1)
+		(body_style 1)
+		(exclude_from_sim no)
+		(in_bom yes)
+		(on_board yes)
+		(in_pos_files yes)
+		(dnp no)
+		(fields_autoplaced yes)
+		(property "Reference" "#PWR023"
+			(at 557.53 43.18 0)
+			(hide yes)
+			(show_name no)
+			(do_not_autoplace no)
+			(effects
+				(font
+					(size 1.27 1.27)
+				)
+			)
+		)
+		(property "Value" "GND"
+			(at 554.99 43.1799 90)
+			(show_name no)
+			(do_not_autoplace no)
+			(effects
+				(font
+					(size 1.27 1.27)
+				)
+				(justify right)
+			)
+		)
+		(property "Footprint" ""
+			(at 551.18 43.18 0)
+			(hide yes)
+			(show_name no)
+			(do_not_autoplace no)
+			(effects
+				(font
+					(size 1.27 1.27)
+				)
+			)
+		)
+		(property "Datasheet" ""
+			(at 551.18 43.18 0)
+			(hide yes)
+			(show_name no)
+			(do_not_autoplace no)
+			(effects
+				(font
+					(size 1.27 1.27)
+				)
+			)
+		)
+		(property "Description" "Power symbol creates a global label with name \"GND\" , ground"
+			(at 551.18 43.18 0)
+			(hide yes)
+			(show_name no)
+			(do_not_autoplace no)
+			(effects
+				(font
+					(size 1.27 1.27)
+				)
+			)
+		)
+		(pin "1"
+		)
+		(instances
+			(project "Picopede"
+				(path "/4d566cad-fdcf-4087-b2b1-2acaa8d49b4f"
+					(reference "#PWR023")
+					(unit 1)
+				)
+			)
+		)
+	)
+	(symbol
 		(lib_id "power:+5VD")
 		(at 97.79 38.1 0)
@@
 		(dnp no)
 		(fields_autoplaced yes)
-		(property "Reference" "J4"
+		(property "Reference" "J1"
 			(at 46.99 31.75 0)
 			(show_name no)
@@
 			(project "Picopede"
 				(path "/4d566cad-fdcf-4087-b2b1-2acaa8d49b4f"
-					(reference "J4")
+					(reference "J1")
 					(unit 1)
 				)
@@
 		(in_pos_files yes)
 		(dnp no)
-		(property "Reference" "C23"
+		(property "Reference" "C5"
 			(at 33.401 148.6916 0)
 			(show_name no)
@@
 			(project "Picopede"
 				(path "/4d566cad-fdcf-4087-b2b1-2acaa8d49b4f"
-					(reference "C23")
+					(reference "C5")
 					(unit 1)
 				)
@@
 		(in_pos_files yes)
 		(dnp no)
-		(property "Reference" "C24"
+		(property "Reference" "C1"
 			(at 76.581 152.5016 0)
 			(show_name no)
@@
 			(project "Picopede"
 				(path "/4d566cad-fdcf-4087-b2b1-2acaa8d49b4f"
-					(reference "C24")
+					(reference "C1")
 					(unit 1)
 				)
@@
 		(dnp no)
 		(fields_autoplaced yes)
-		(property "Reference" "J4"
+		(property "Reference" "J5"
 			(at 544.83 148.5899 0)
 			(show_name no)
@@
 			(project "Picopede"
 				(path "/4d566cad-fdcf-4087-b2b1-2acaa8d49b4f"
-					(reference "J4")
+					(reference "J5")
 					(unit 1)
 				)
@@
 		(dnp no)
 		(fields_autoplaced yes)
-		(property "Reference" "J3"
+		(property "Reference" "J4"
 			(at 500.38 148.5899 0)
 			(show_name no)
@@
 			(project "Picopede"
 				(path "/4d566cad-fdcf-4087-b2b1-2acaa8d49b4f"
-					(reference "J3")
+					(reference "J4")
 					(unit 1)
 				)
@@
 		(in_pos_files yes)
 		(dnp no)
-		(fields_autoplaced yes)
-		(property "Reference" "J1"
-			(at 499.11 76.1999 0)
+		(property "Reference" "J2"
+			(at 496.316 31.75 0)
 			(show_name no)
 			(do_not_autoplace no)
@@
 		)
 		(property "Value" "Conn_01x32"
-			(at 499.11 78.7399 0)
+			(at 491.49 33.782 0)
 			(show_name no)
 			(do_not_autoplace no)
@@
 			(project "Picopede"
 				(path "/4d566cad-fdcf-4087-b2b1-2acaa8d49b4f"
-					(reference "J1")
+					(reference "J2")
 					(unit 1)
 				)
@@
 		(dnp no)
 		(fields_autoplaced yes)
-		(property "Reference" "J2"
-			(at 525.78 76.1999 0)
+		(property "Reference" "J3"
+			(at 528.32 31.75 0)
 			(show_name no)
 			(do_not_autoplace no)
@@
 					(size 1.27 1.27)
 				)
-				(justify left)
 			)
 		)
 		(property "Value" "Conn_01x32"
-			(at 525.78 78.7399 0)
+			(at 528.32 34.29 0)
 			(show_name no)
 			(do_not_autoplace no)
@@
 					(size 1.27 1.27)
 				)
-				(justify left)
 			)
 		)
@@
 			(project "Picopede"
 				(path "/4d566cad-fdcf-4087-b2b1-2acaa8d49b4f"
-					(reference "J2")
+					(reference "J3")
 					(unit 1)
 				)
